File: A1200KB.kicad_pcb (KiCad board)
At the start: 2 copper layers, 449.2 x 124.3 mm, 107 parts, among them J1 Conn_01x32_Female, K1 ESC, K10 F9, K11 F10, K12 TILDE, K13 1, K14 2, K15 3, K16 4, K17 5, K18 6, K19 7, K2 F1, K20 8, K21 9, K22 0, K23 MINUS, K24 PLUS, K25 PIPE, K26 BS, K27 DEL, K28 HELP, K29 NUM_(, K3 F2, K30 NUM_), K31 NUM_DIV, K32 NUM_MULT, K33 TAB, K34 Q, K35 W, K36 E, K37 R, K38 T, K39 Y, K4 F3, K40 U, K41 I, K42 O, K43 P, K44 L.CURLY, K45 R.CURLY, K46 RETURN, K47 NUM_7, K48 NUM_8, K49 NUM_9, K5 F4, K50 NUM_MINUS, K51 CTRL, K52 CAPSLOCK, K53 A, K54 S, K55 D, K56 F, K57 G, K58 H, K59 J, K6 F5, K60 K, K61 L, K62 COLON, K63 ", K64 R.BLANK, K65 UP, K66 NUM_4, K67 NUM_5, K68 NUM_6, K69 NUM_PLUS, K7 F6, K70 L.SHIFT, K71 L.BLANK, K72 Z, K73 X, K74 C, K75 V, K76 B, K77 N, K78 M, K79 R.CROC, K8 F7, K80 L.CROC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

Commit message: Now has the AmigaComponents.lib dependancy
Parts:
- removed BK1, BK2: BLANK, MX_Alps_Hybrid:MXOnly-1U-NoLED
- removed REF** (x7): MountingHole_3.2mm_M3, MountingHole:MountingHole_3.2mm_M3
- removed REF**: ALT-9U, MX_Alps_Hybrid:MX-9U
- added H1: MountingHole_Pad, MountingHole:MountingHole_3mm_Pad, F.Cu at (76.0, 128.7)
- added H11: MountingHole_Pad, MountingHole:MountingHole_3mm_Pad, F.Cu at (345.3, 180.5)
- added H12: MountingHole_Pad, MountingHole:MountingHole_3mm_Pad, F.Cu at (354.8, 137.6)
- added H13: MountingHole_Pad, MountingHole:MountingHole_3mm_Pad, F.Cu at (366.7, 242.4)
- added H14: MountingHole_Pad, MountingHole:MountingHole_3mm_Pad, F.Cu at (390.5, 194.8)
- added H15: MountingHole_Pad, MountingHole:MountingHole_3mm_Pad, F.Cu at (438.1, 242.4)
- added H17: MountingHole_Pad, MountingHole:MountingHole_3mm_Pad, F.Cu at (502.4, 216.2)
- added H18: MountingHole_Pad, MountingHole:MountingHole_3mm_Pad, F.Cu at (519.3, 128.7)
- added H19: MountingHole_Pad, MountingHole:MountingHole_3mm_Pad, F.Cu at (519.3, 256.1)
- added H2: MountingHole_Pad, MountingHole:MountingHole_3mm_Pad, F.Cu at (76.0, 256.0)
- added H3: MountingHole_Pad, MountingHole:MountingHole_3mm_Pad, F.Cu at (116.7, 154.3)
- added H5: MountingHole_Pad, MountingHole:MountingHole_3mm_Pad, F.Cu at (192.8, 242.4)
- added H6: MountingHole_Pad, MountingHole:MountingHole_3mm_Pad, F.Cu at (197.1, 157.1)
- added H7: MountingHole_Pad, MountingHole:MountingHole_3mm_Pad, F.Cu at (207.2, 195.0)
- added H8: MountingHole_Pad, MountingHole:MountingHole_3mm_Pad, F.Cu at (226.2, 137.7)
- added H9: MountingHole_Pad, MountingHole:MountingHole_3mm_Pad, F.Cu at (250.0, 242.4)
- added K97: MENU, RetroBitLab:SW_Cherry_MX1A_1.00u_PCB_3d, F.Cu at (295.1, 249.8)
- added K98: SUPER, RetroBitLab:SW_Cherry_MX1A_1.00u_PCB_3d, F.Cu at (142.6, 249.9)
- added K99: SPACE 9U, RetroBitLab:SW_Cherry_MX1A_9u_PCB_3d, F.Cu at (218.9, 249.9)
- added U1: STM32F401-DK, RetroBitLab:STM32F401-DK, B.Cu at (409.8, 154.7)
- J1: footprint Connector_FFC-FPC:FFC-1.25mm-RA-5204403245 -> RetroBitLab:MOLEX-FFC-1.25mm-RA-52044-3245
- K1, K13, K14, K15, K16, K17, K18, K19, K20, K21, K22, K23, K24, K25, K26, K29, K30, K31, K32, K34, K35, K36, K37, K38, K39, K40, K41, K42, K43, K44, K45, K47, K48, K49, K50, K53, K54, K55, K56, K57, K58, K59, K60, K61, K62, K63, K64, K65, K66, K67, K68, K69, K71, K72, K73, K74, K75, K76, K77, K78, K79, K80, K81, K83, K84, K85, K86, K87, K88, K96: footprint MX_Alps_Hybrid:MXOnly-1U-NoLED -> RetroBitLab:SW_Cherry_MX1A_1.00u_PCB_3d
- K10, K11, K2, K3, K4, K5, K51, K6, K7, K8, K9, K90, K91, K93, K94: footprint MX_Alps_Hybrid:MXOnly-1.25U-NoLED -> RetroBitLab:SW_Cherry_MX1A_1.25u_PCB_3d
- K12, K27, K28: footprint MX_Alps_Hybrid:MXOnly-1.5U-NoLED -> RetroBitLab:SW_Cherry_MX1A_1.50u_PCB_3d
- K33: footprint MX_Alps_Hybrid:MXOnly-2U-NoLED -> RetroBitLab:SW_Cherry_MX1A_1.00u_PCB_3d
- K46: footprint MX_Alps_Hybrid:MXOnly-ISO -> RetroBitLab:SW_Cherry_MX1A_ISOEnter_PCB_3d
- K52: footprint MX_Alps_Hybrid:MXOnly-1U -> RetroBitLab:MXOnly-1U
- K70: footprint MX_Alps_Hybrid:MXOnly-1.75U-NoLED -> RetroBitLab:SW_Cherry_MX1A_1.75u_PCB_3d
- K82: footprint MX_Alps_Hybrid:MXOnly-2.75U-NoLED -> RetroBitLab:SW_Cherry_MX1A_2.75u_PCB_3d
- K89: footprint MX_Alps_Hybrid:MXOnly-2U-NoLED -> RetroBitLab:SW_Cherry_MX1A_2.00u_Vertical_PCB_3d
- K92: value SPACE -> SPACE 7U; footprint MX_Alps_Hybrid:MXOnly-7U-NoLED -> RetroBitLab:MXOnly-7U-NoSwitch
- K95: footprint MX_Alps_Hybrid:MXOnly-2U-NoLED -> RetroBitLab:SW_Cherry_MX1A_2.00u_PCB_3d
- moved K13 449.9 mm to (406.8, 344.2)
- moved K1 434.1 mm to (217.8, 426.3)
- moved K52 408.1 mm to (261.6, 451.6)
- moved K11 403.6 mm to (170.2, 425.2)
- moved K71 395.9 mm to (386.6, 344.2)
- moved K72 385.9 mm to (406.8, 324.0)
- moved K53 385.7 mm to (243.9, 446.5)
- moved K17 385.1 mm to (183.3, 446.5)
- moved K20 381.1 mm to (163.1, 445.4)
- moved K33 380.7 mm to (311.7, 345.5)
- moved K18 380.3 mm to (142.9, 445.4)
- moved K9 379.4 mm to (145.3, 406.1)
- moved K10 378.0 mm to (170.2, 405.0)
- moved K73 374.6 mm to (284.3, 446.5)
- moved K21 373.7 mm to (359.2, 406.1)
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Routing:
- net /15: track 634.3 -> 0.00 mm, vias 2 -> 0
- net /4: track 598.3 -> 0.00 mm, vias 1 -> 0
- net /17: track 594.1 -> 0.00 mm, vias 1 -> 0
- net /3: track 556.4 -> 0.00 mm, vias 2 -> 0
- net /2: track 549.9 -> 0.00 mm, vias 3 -> 0
- net /18: track 538.4 -> 0.00 mm, vias 1 -> 0
- net /16: track 529.9 -> 0.00 mm, vias 3 -> 0
- net /19: track 515.6 -> 0.00 mm, vias 2 -> 0
- net /1: track 488.1 -> 0.00 mm, vias 3 -> 0
- net /20: track 476.7 -> 0.00 mm, vias 2 -> 0
- net /30: track 462.4 -> 0.00 mm, vias 1 -> 0
- net /7: track 456.0 -> 0.00 mm
- net /24: track 440.6 -> 0.00 mm, vias 1 -> 0
- net /27: track 434.9 -> 0.00 mm, vias 3 -> 0
- net /29: track 423.4 -> 0.00 mm, vias 1 -> 0
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Other:
- board size 449.2 x 124.3 mm -> 449.3 x 141.4 mm
- board text removed: "195, 115"
- board text removed: "295, 115"
- board text removed: "370, 115"
- board text removed: "442, 87"
- board text removed: "7, 115"
- board text removed: "7, 25"
- board text removed: "95, 115"
- board text removed: "A1200KB"
- board text removed: "December 2019"
- board text removed: "Rev.3"
- board text removed: "aeberbach"
- board text removed: "grayunicorn.com"

Commit message: The ISO Enter here, must have rotated Cherry MX switch by 180 degrees
Parts:
- added H16: MountingHole_Pad, MountingHole:MountingHole_3mm_Pad, F.Cu at (47.2, 180.8)
- K46: footprint RetroBitLab:SW_Cherry_MX1A_ISOEnter_PCB_3d -> RetroBitLab:SW_Cherry_MX1A_ISOEnter_Rotated_PCB_3d
- moved K28 265.5 mm to (418.9, 173.7), turned to 180 degrees
- moved K46 222.3 mm to (359.7, 192.1)
- moved K70 161.6 mm to (87.9, 230.8), turned to 180 degrees
- moved K82 53.4 mm to (340.3, 230.8), turned to 180 degrees

Commit message: Added MCU controller sheet page
Parts:
- removed H16: MountingHole_Pad, MountingHole:MountingHole_3mm_Pad
- moved U1 4.86 mm to (414.6, 154.4)
