File: A1200KB.kicad_pcb (KiCad board)
At the start: 2 copper layers, 449.3 x 141.4 mm, 117 parts, among them J1 Conn_01x32_Female, K1 ESC, K10 F9, K11 F10, K12 TILDE, K13 1, K14 2, K15 3, K16 4, K17 5, K18 6, K19 7, K2 F1, K20 8, K21 9, K22 0, K23 MINUS, K24 PLUS, K25 PIPE, K26 BS, K27 DEL, K28 HELP, K29 NUM_(, K3 F2, K30 NUM_), K31 NUM_DIV, K32 NUM_MULT, K33 TAB, K34 Q, K35 W, K36 E, K37 R, K38 T, K39 Y, K4 F3, K40 U, K41 I, K42 O, K43 P, K44 L.CURLY, K45 R.CURLY, K46 RETURN, K47 NUM_7, K48 NUM_8, K49 NUM_9, K5 F4, K50 NUM_MINUS, K51 CTRL, K52 CAPSLOCK, K53 A, K54 S, K55 D, K56 F, K57 G, K58 H, K59 J, K6 F5, K60 K, K61 L, K62 COLON, K63 ", K64 R.BLANK, K65 UP, K66 NUM_4, K67 NUM_5, K68 NUM_6, K69 NUM_PLUS, K7 F6, K70 L.SHIFT, K71 L.BLANK, K72 Z, K73 X, K74 C, K75 V, K76 B, K77 N, K78 M, K79 R.CROC, K8 F7, K80 L.CROC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

Commit message: Updated from AEBERBACH GitHub repo
Parts:
- removed H1, H11, H12, H13, H14, H15, H17, H18, H19, H2, H3, H5, H6, H7, H8, H9: MountingHole_Pad, MountingHole:MountingHole_3mm_Pad
- removed K97: MENU, RetroBitLab:SW_Cherry_MX1A_1.00u_PCB_3d
- removed K98: SUPER, RetroBitLab:SW_Cherry_MX1A_1.00u_PCB_3d
- removed K99: SPACE 9U, RetroBitLab:SW_Cherry_MX1A_9u_PCB_3d
- removed U1: STM32F401-DK, RetroBitLab:STM32F401-DK
- added REF**: MountingHole_3.2mm_M3, MountingHole:MountingHole_3.2mm_M3, F.Cu at (465.4, 137.0)
- added REF**: MountingHole_3.2mm_M3, MountingHole:MountingHole_3.2mm_M3, F.Cu at (57.9, 169.0)
- added REF**: MountingHole_3.2mm_M3, MountingHole:MountingHole_3.2mm_M3, F.Cu at (57.8, 100.7)
- added REF**: ALT-9U, MX_Alps_Hybrid:MX-9U, F.Cu at (198.2, 190.4)
- J1: footprint RetroBitLab:MOLEX-FFC-1.25mm-RA-52044-3245 -> Connector_FFC-FPC:FFC-1.25mm-RA-5204403245
- K1, K13, K14, K15, K16, K17, K18, K19, K20, K21, K22, K23, K24, K25, K26, K29, K30, K31, K32, K34, K35, K36, K37, K38, K39, K40, K41, K42, K43, K44, K45, K47, K48, K49, K50, K53, K54, K55, K56, K57, K58, K59, K60, K61, K62, K63, K64, K65, K66, K67, K68, K69, K71, K72, K73, K74, K75, K76, K77, K78, K79, K80, K81, K83, K84, K85, K86, K87, K88, K96: footprint RetroBitLab:SW_Cherry_MX1A_1.00u_PCB_3d -> MX_Alps_Hybrid:MXOnly-1U-NoLED
- K10, K11, K2, K3, K4, K5, K51, K6, K7, K8, K9, K90, K91, K93, K94: footprint RetroBitLab:SW_Cherry_MX1A_1.25u_PCB_3d -> MX_Alps_Hybrid:MXOnly-1.25U-NoLED
- K12, K27, K28: footprint RetroBitLab:SW_Cherry_MX1A_1.50u_PCB_3d -> MX_Alps_Hybrid:MXOnly-1.5U-NoLED
- K33: footprint RetroBitLab:SW_Cherry_MX1A_1.00u_PCB_3d -> MX_Alps_Hybrid:MXOnly-2U-NoLED
- K46: footprint RetroBitLab:SW_Cherry_MX1A_ISOEnter_Rotated_PCB_3d -> MX_Alps_Hybrid:MXOnly-ISO
- K52: footprint RetroBitLab:MXOnly-1U -> MX_Alps_Hybrid:MXOnly-1U
- K70: footprint RetroBitLab:SW_Cherry_MX1A_1.75u_PCB_3d -> MX_Alps_Hybrid:MXOnly-1.75U-NoLED
- K82: footprint RetroBitLab:SW_Cherry_MX1A_2.75u_PCB_3d -> MX_Alps_Hybrid:MXOnly-2.75U-NoLED
- K89: footprint RetroBitLab:SW_Cherry_MX1A_2.00u_Vertical_PCB_3d -> MX_Alps_Hybrid:MXOnly-2U-NoLED
- K92: value SPACE 7U -> SPACE; footprint RetroBitLab:MXOnly-7U-NoSwitch -> MX_Alps_Hybrid:MXOnly-7U-NoLED
- K95: footprint RetroBitLab:SW_Cherry_MX1A_2.00u_PCB_3d -> MX_Alps_Hybrid:MXOnly-2U-NoLED
- moved K13 392.1 mm to (89.3, 114.2)
- moved K1 375.1 mm to (60.9, 85.6)
- moved K11 369.5 mm to (315.4, 85.4)
- moved K52 347.8 mm to (84.5, 152.3)
- moved K9 343.3 mm to (267.6, 85.4)
- moved K10 341.9 mm to (291.5, 85.4)
- moved K71 339.7 mm to (94.1, 171.3)
- moved K20 336.5 mm to (222.7, 114.2)
- moved K18 333.8 mm to (184.6, 114.2)
- moved K69 333.6 mm to (488.7, 152.2)
- moved K49 333.4 mm to (469.7, 133.1)
- moved K17 332.8 mm to (165.5, 114.2)
- moved K72 330.9 mm to (113.2, 171.3)
- moved K53 326.0 mm to (103.5, 152.3)
- moved K33 321.5 mm to (70.3, 133.2)
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Routing:
- net /4: track 0.00 -> 595.0 mm, vias 0 -> 1
- net /15: track 0.00 -> 551.7 mm, vias 0 -> 2
- net /16: track 0.00 -> 538.7 mm, vias 0 -> 4
- net /17: track 0.00 -> 514.7 mm, vias 0 -> 3
- net /19: track 0.00 -> 500.9 mm, vias 0 -> 3
- net /3: track 0.00 -> 493.1 mm, vias 0 -> 2
- net /18: track 0.00 -> 483.4 mm, vias 0 -> 3
- net /30: track 0.00 -> 480.3 mm, vias 0 -> 3
- net /7: track 0.00 -> 454.3 mm, vias 0 -> 1
- net /20: track 0.00 -> 453.8 mm, vias 0 -> 2
- net /27: track 0.00 -> 449.1 mm, vias 0 -> 3
- net /21: track 0.00 -> 446.5 mm, vias 0 -> 7
- net /2: track 0.00 -> 427.2 mm, vias 0 -> 2
- net /29: track 0.00 -> 422.5 mm, vias 0 -> 2
- net /24: track 0.00 -> 421.4 mm, vias 0 -> 3
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Other:
- board size 449.3 x 141.4 mm -> 450 x 125 mm
- board text added: "+"
- board text added: "7,103"
- board text added: "7,38"
- board text added: "7,7"
- board text added: "A1200KB"
- board text added: "July 2021"
- board text added: "Rev.4"
- board text added: "aeberbach"
- board text added: "grayunicorn.com"
